File: myra-sip-interposer.kicad_sch (KiCad schematic)
At the start: 32 parts, among them U1 FT231XQ-R, U2 MB85RS1MTPW-G_WLP, U3 NCP177AMX330TCG, U4 STM32G491REI6, U5 Myra-231F1F08_CUSTOM_mirrored, Y1 Resonator_32.768kHz_ECX-1210, Y2 Oscillator_8MHz_ECS_1612MV

Commit message: [#63584] Rename project to Myra SiP Interposer
Parts:
- U5: GitHub https://github.com/antmicro/myra-sip -> https://github.com/antmicro/myra-sip-interposer
Other:
- title: MYRA SiP -> Myra SiP Interposer
